File: BlastersRev2.sch (KiCad schematic (older format))
At the start: 61 parts, among them U1 ProMicro

Commit message: All components placed
Parts:
- D1, D10, D11, D12, D13, D14, D15, D16, D17, D18, D19, D2, D20, D21, D22, D23, D24, D25, D26, D27, D28, D29, D3, D30, D4, D5, D6, D7, D8, D9: footprint Keebio-Parts:Diode -> Keebio-Parts:Diode-dual
- MX1, MX10, MX11, MX12, MX13, MX14, MX15, MX16, MX17, MX18, MX19, MX2, MX20, MX21, MX22, MX23, MX24, MX25, MX26, MX27, MX28, MX29, MX3, MX30, MX4, MX5, MX6, MX7, MX8, MX9: footprint keyswitches:MX_reversible -> Keebio-Parts:Hybrid_PCB_100H_Dual_hole

Commit message: Done!
Parts:
- added J1: AudioJack4_Ground, Keebio-Parts:TRRS-PJ-320A-dual, symbol Connector:AudioJack4_Ground
- added JP1: Jumper, Jumper:SolderJumper-2_P1.3mm_Open_Pad1.0x1.5mm, symbol Device:Jumper
- added MH1: MountingHole_Pad, MountingHole:MountingHole_2.2mm_M2_DIN965_Pad, symbol Mechanical:MountingHole_Pad
Connections:
- net Col0: now also U1.18 (F6)
- net Col1: now also U1.17 (F7)
- net Col2: now also U1.16 (B1)
- net Col3: now also U1.19 (F5)
- net Col4: now also U1.7 (D4)
- net Col5: now also U1.6 (SDA)
- net Col6: now also U1.5 (SCL)
- net Row0: now also U1.9 (D7)
- net Row1: now also U1.15 (B3)
- net Row2: now also U1.14 (B2)
- net Row3: now also U1.13 (B6)
- net Row4: now also U1.12 (B5)
- net Comm: now reaches U1.20 (F4)
- net Comm: now also J1.R2
- net CommVcc: now reaches U1.21 (VCC)
- net CommVcc: now also J1.T
- net CommGnd: now reaches U1.23 (GND)
- net CommGnd: now also J1.S
- net RGBGnd: now reaches U1.3 (GND)
- net RGBCommBreakout: now reaches U1.8 (C6)
- net RGBCommBreakout: now also JP1.1, MH1.1
- new net RGBTrrs: J1.R1, JP1.2
Changed lines of the file:
@@
 EESchema Schematic File Version 4
+LIBS:BlastersRev2-cache
 EELAYER 26 0
 EELAYER END
@@
 Text GLabel 9150 1500 1    50   Input ~ 0
 Col6
+$Comp
+L Connector:AudioJack4_Ground J1
+U 1 1 5D080F1A
+P 2850 3900
+F 0 "J1" H 2816 4242 50  0000 C CNN
+F 1 "AudioJack4_Ground" H 2816 4151 50  0000 C CNN
+F 2 "Keebio-Parts:TRRS-PJ-320A-dual" H 2850 3900 50  0001 C CNN
+F 3 "~" H 2850 3900 50  0001 C CNN
+	1    2850 3900
+	1    0    0    -1
+$EndComp
+Text GLabel 3050 3800 2    50   Input ~ 0
+CommGnd
+Text GLabel 3050 4100 2    50   Input ~ 0
+CommVcc
+Text GLabel 3050 3900 2    50   Input ~ 0
+Comm
+Text GLabel 3050 4000 2    50   Input ~ 0
+RGBTrrs
+Text GLabel 3800 2000 2    50   Input ~ 0
+CommGnd
+Text GLabel 3800 2300 2    50   Input ~ 0
+Comm
+Text GLabel 1850 2650 3    50   Input ~ 0
+RGBJumper
+Text GLabel 4350 2250 3    50   Input ~ 0
+CommVcc
+Text GLabel 4350 2150 1    50   Input ~ 0
+RGBVcc
+Wire Wire Line
+	3800 2200 4350 2200
+Wire Wire Line
+	4350 2150 4350 2200
+Connection ~ 4350 2200
+Wire Wire Line
+	4350 2200 4350 2250
+Text GLabel 2400 2100 0    50   Input ~ 0
+RGBGnd
+Text GLabel 1850 2550 1    50   Input ~ 0
+RGBCommBreakout
+Wire Wire Line
+	1850 2550 1850 2600
+Wire Wire Line
+	1850 2600 2400 2600
+Connection ~ 1850 2600
+Wire Wire Line
+	1850 2600 1850 2650
+$Comp
+L Mechanical:MountingHole_Pad MH1
+U 1 1 5D09799C
+P 4050 3800
+F 0 "MH1" H 4150 3851 50  0000 L CNN
+F 1 "MountingHole_Pad" H 4150 3760 50  0000 L CNN
+F 2 "MountingHole:MountingHole_2.2mm_M2_DIN965_Pad" H 4050 3800 50  0001 C CNN
+F 3 "~" H 4050 3800 50  0001 C CNN
+	1    4050 3800
+	1    0    0    -1
+$EndComp
+Text GLabel 4050 3900 3    50   Input ~ 0
+RGBCommBreakout
+$Comp
+L Device:Jumper JP1
+U 1 1 5D097F50
+P 3200 5050
+F 0 "JP1" H 3200 5314 50  0000 C CNN
+F 1 "Jumper" H 3200 5223 50  0000 C CNN
+F 2 "Jumper:SolderJumper-2_P1.3mm_Open_Pad1.0x1.5mm" H 3200 5050 50  0001 C CNN
+F 3 "~" H 3200 5050 50  0001 C CNN
+	1    3200 5050
+	1    0    0    -1
+$EndComp
+Text GLabel 2900 5050 0    50   Input ~ 0
+RGBJumper
+Text GLabel 3500 5050 2    50   Input ~ 0
+RGBTrrs
+Text GLabel 2400 2700 0    50   Input ~ 0
+Row0
+Text GLabel 3800 2400 2    50   Input ~ 0
+Col3
+Text GLabel 2400 2500 0    50   Input ~ 0
+Col4
+Text GLabel 2400 2300 0    50   Input ~ 0
+Col6
+Text GLabel 2400 2400 0    50   Input ~ 0
+Col5
+Text GLabel 3800 2700 2    50   Input ~ 0
+Col2
+Text GLabel 3800 2600 2    50   Input ~ 0
+Col1
+Text GLabel 3800 2500 2    50   Input ~ 0
+Col0
+Text GLabel 3800 2800 2    50   Input ~ 0
+Row1
+Text GLabel 3800 2900 2    50   Input ~ 0
+Row2
+Text GLabel 3800 3000 2    50   Input ~ 0
+Row3
+Text GLabel 2400 3000 0    50   Input ~ 0
+Row4
 $EndSCHEMATC
